Commit message: added controller and joints to urdf file

File: PiCar-X/picarx_description/urdf/picarx/picarx.urdf (robot description, URDF)
Before this commit: robot picarx, 8 links, 7 joints
Links:
- added link picarx_steer_bar, mass 1; visual box size=0.01 0.099 0.003
- added link picarx_steer_bar_screw_left, mass 1; visual cylinder length=0.005 radius=0.005
- added link picarx_steer_bar_screw_right, mass 1; visual cylinder length=0.005 radius=0.005
- added link picarx_steer_servo, mass 1; visual cylinder length=0.005 radius=0.005
Joints:
- added joint base_link_JOINT_steer_servo: type fixed, parent base_link, child picarx_steer_servo, origin xyz=0.139   0.0  0.0485 rpy=0  0  0
- added joint picarx_steer_fl_JOINT_steer_bar_screw_fl: type fixed, parent picarx_steer_fl, child picarx_steer_bar_screw_left
- added joint picarx_steer_fr_JOINT_steer_bar_screw_right: type fixed, parent picarx_steer_fr, child picarx_steer_bar_screw_right
- added joint steer_bar_screw_left_JOINT_steer_bar: type fixed, parent picarx_steer_bar, child picarx_steer_bar_screw_left, origin xyz=0.0   0.0235  0.00 rpy=0  0  0
- added joint steer_bar_screw_right_JOINT_steer_bar: type fixed, parent picarx_steer_bar, child picarx_steer_bar_screw_right, origin xyz=0.0   -0.0235 0.00 rpy=0  0  0
- added joint steer_servo_JOINT_steer_bar: type prismatic, parent picarx_steer_servo, child picarx_steer_bar, origin xyz=0.02   0.0  0.0 rpy=0  0  0, axis 0  1  0, limit lower=-1.5708 upper=1.5708 effort=1.0 velocity=1.0
- joint base_link_JOINT_steer_fl: origin xyz=0.137  0.049  0.029 rpy=0  0  0 -> xyz=0.139  0.048  0.04 rpy=0  0  0
- joint base_link_JOINT_steer_fr: origin xyz=0.137   -0.04999  0.029 rpy=0  0  0 -> xyz=0.139   -0.048  0.04 rpy=0  0  0
- joint joint_wheel_left: origin xyz=-0.01949  0.06926  0.03808 rpy=1.5708  0      0 -> xyz=-0.0195  0.065  0.04 rpy=1.5708  0      0
- joint joint_wheel_right: origin xyz=-0.0195  -0.06925  0.03808 rpy=1.5708  0      0 -> xyz=-0.0195  -0.065  0.04 rpy=1.5708  0      0
- joint picarx_steer_fl_JOINT_FrontLeft: origin xyz=0.00542  0.01983  0.00908 rpy=1.5708  0      0 -> xyz=0.00542  0.01983  -0.0025 rpy=1.5708  0      0; type revolute -> continuous
- joint picarx_steer_fr_JOINT_FrontRight: origin xyz=0.00542 -0.01816  0.00908 rpy=1.5708  0      0 -> xyz=0.00542 -0.01816  -0.0025 rpy=1.5708  0      0; type revolute -> continuous

Commit message: backup with steering bars

File: PiCar-X/picarx_description/urdf/picarx/picarx.urdf (robot description, URDF)
Before this commit: robot picarx, 12 links, 13 joints
Links:
- removed link base_footprint
- removed link base_link
- removed link picarx_WheelFrontLeft
- removed link picarx_WheelFrontRight
- removed link picarx_steer_bar
- removed link picarx_steer_bar_screw_left
- removed link picarx_steer_bar_screw_right
- removed link picarx_steer_servo
- added link chassis, mass 1; collision mesh filename=package://picarx_description/meshes/Chassis.dae scale=1 1 1; visual mesh filename=package://picarx_description/meshes/Chassis.dae scale=1 1 1
- added link picarx_steer_bar_l, mass 1; collision box size=0.01 0.043 0.003; visual box size=0.01 0.043 0.003
- added link picarx_steer_bar_r, mass 1; collision box size=0.01 0.043 0.003; visual box size=0.01 0.043 0.003
- added link world
- link left_wheel: geometry collision mesh filename=package://picarx_description/meshes/WheelRearLeft.dae scale=1 1 1; visual mesh filename=package://picarx_description/meshes/WheelRearLeft.dae scale=1 1 1
- link picarx_steer_fl: geometry collision box size=0.02 0.01 0.024; visual box size=0.02 0.01 0.024
- link picarx_steer_fr: geometry collision box size=0.02 0.01 0.024; visual box size=0.02 0.01 0.024
- link right_wheel: geometry collision mesh filename=package://picarx_description/meshes/WheelRearRight.dae scale=1 1 1; visual mesh filename=package://picarx_description/meshes/WheelRearRight.dae scale=1 1 1
Joints:
- removed joint base_footprint_joint
- removed joint base_link_JOINT_steer_fl
- removed joint base_link_JOINT_steer_fr
- removed joint base_link_JOINT_steer_servo
- removed joint picarx_steer_fl_JOINT_FrontLeft
- removed joint picarx_steer_fl_JOINT_steer_bar_screw_fl
- removed joint picarx_steer_fr_JOINT_FrontRight
- removed joint picarx_steer_fr_JOINT_steer_bar_screw_right
- removed joint steer_bar_screw_left_JOINT_steer_bar
- removed joint steer_bar_screw_right_JOINT_steer_bar
- removed joint steer_servo_JOINT_steer_bar
- added joint chassis_to_world: type fixed, parent world, child chassis
- added joint steer_left: type continuous, parent chassis, child picarx_steer_fl, origin xyz=0.13   0.043  0.0395 rpy=0  0  0, axis 0 0 1
- added joint steer_right: type continuous, parent chassis, child picarx_steer_fr, origin xyz=0.13   -0.043  0.0395 rpy=0  0  0, axis 0 0 1
- added joint steerbar_left: type continuous, parent picarx_steer_fl, child picarx_steer_bar_l, origin xyz=0.01999999  0  0 rpy=0 0 0, axis 0 0 1
- added joint steerbar_right: type continuous, parent picarx_steer_fr, child picarx_steer_bar_r, origin xyz=0.01999999   0  0 rpy=0.0 0 0, axis 0 0 1
- joint joint_wheel_left: child right_wheel -> left_wheel; limit lower=-1.79769e+308 upper=1.79769e+308 effort=1.0 velocity=1.0 -> (none); origin xyz=-0.0195  0.065  0.04 rpy=1.5708  0      0 -> xyz=0.0   0.063  0.04 rpy=1.5708  0 0; parent base_link -> chassis
- joint joint_wheel_right: child left_wheel -> right_wheel; limit lower=-1.79769e+308 upper=1.79769e+308 effort=1.0 velocity=1.0 -> (none); origin xyz=-0.0195  -0.065  0.04 rpy=1.5708  0      0 -> xyz=0.0   -0.063  0.04 rpy=1.5708 0      0; parent base_link -> chassis
