Commit message: moved gazebo packages to simulation folder and added Dockerfile

File: PiCar-X/simulation/picarx_description/urdf/picarx/picarx.urdf (robot description, URDF)
Before this commit: robot picarx, 8 links, 7 joints
Links:
- removed link picarx_steer_bar_l
- removed link picarx_steer_bar_r
- added link picarx_WheelFrontLeft, mass 1; collision mesh filename=package://picarx_description/meshes/WheelFrontLeft.dae scale=1 1 1; visual mesh filename=package://picarx_description/meshes/WheelFrontLeft.dae scale=1 1 1
- added link picarx_WheelFrontRight, mass 1; collision mesh filename=package://picarx_description/meshes/WheelFrontRight.dae scale=1 1 1; visual mesh filename=package://picarx_description/meshes/WheelFrontRight.dae scale=1 1 1
Joints:
- removed joint steerbar_left
- removed joint steerbar_right
- added joint front_left_wheel: type continuous, parent picarx_steer_fl, child picarx_WheelFrontLeft, origin xyz=0.0 0.015 -0.0025 rpy=0 0 0, axis 0  0  1
- added joint front_right_wheel: type continuous, parent picarx_steer_fr, child picarx_WheelFrontRight, origin xyz=0.0 -0.015 -0.0025 rpy=0 0 0, axis 0  0  1
- joint joint_wheel_left: origin xyz=0.0   0.063  0.04 rpy=1.5708  0 0 -> xyz=0.0   0.063  0.0375 rpy=1.5708  0 0
- joint joint_wheel_right: origin xyz=0.0   -0.063  0.04 rpy=1.5708 0      0 -> xyz=0.0   -0.063  0.0375 rpy=1.5708 0      0
- joint steer_left: origin xyz=0.13   0.043  0.0395 rpy=0  0  0 -> xyz=0.135   0.048  0.04 rpy=0  0  0
- joint steer_right: origin xyz=0.13   -0.043  0.0395 rpy=0  0  0 -> xyz=0.135   -0.048  0.04 rpy=0  0  0

Commit message: - added emulators and drivers for clutchgears and dcmotor. - First DTP!

File: PiCar-X/simulation/picarx_description/urdf/picarx/picarx.urdf (robot description, URDF)
Before this commit: robot picarx, 8 links, 7 joints
Joints:
- joint steer_left: limit (none) -> lower=-0.698 upper=0.698 effort=10 velocity=1; origin xyz=0.135   0.048  0.04 rpy=0  0  0 -> xyz=0.14   0.048  0.04 rpy=0  0  0; type continuous -> revolute
- joint steer_right: limit (none) -> lower=-0.698 upper=0.698 effort=10 velocity=1; origin xyz=0.135   -0.048  0.04 rpy=0  0  0 -> xyz=0.14   -0.048  0.04 rpy=0  0  0; type continuous -> revolute

Commit message: model has more realistic interia values

File: PiCar-X/simulation/picarx_description/urdf/picarx/picarx.urdf (robot description, URDF)
Before this commit: robot picarx, 8 links, 7 joints
Links:
- link left_wheel: mass 1 -> 0.1; geometry collision mesh filename=package://picarx_description/meshes/WheelRearRight.dae scale=1 1 1; visual mesh filename=package://picarx_description/meshes/WheelRearRight.dae scale=1 1 1
- link picarx_WheelFrontLeft: mass 1 -> 0.025; geometry collision mesh filename=package://picarx_description/meshes/WheelFrontLef.dae scale=1 1 1; visual mesh filename=package://picarx_description/meshes/WheelFrontLeft.dae scale=1 1 1
- link picarx_WheelFrontRight: mass 1 -> 0.025; geometry collision mesh filename=package://picarx_description/meshes/WheelFrontLeft.dae scale=1 1 1; visual mesh filename=package://picarx_description/meshes/WheelFrontLeft.dae scale=1 1 1
- link picarx_steer_fl: mass 1 -> 0.005
- link picarx_steer_fr: mass 1 -> 0.005
- link right_wheel: mass 1 -> 0.1
Joints:
- joint front_left_wheel: origin xyz=0.0 0.015 -0.0025 rpy=0 0 0 -> xyz=0.0 0.005 -0.0045 rpy=-1.5708 0 0
- joint front_right_wheel: origin xyz=0.0 -0.015 -0.0025 rpy=0 0 0 -> xyz=0.0 -0.005 -0.005 rpy=1.5708 0 0
- joint joint_wheel_left: origin xyz=0.0   0.063  0.0375 rpy=1.5708  0 0 -> xyz=0 0.055 0.0326 rpy=-1.5708  0 0
- joint joint_wheel_right: origin xyz=0.0   -0.063  0.0375 rpy=1.5708 0      0 -> xyz=0 -0.055 0.0326 rpy=1.5708  0 0
- joint steer_left: axis 0 0 1 -> (none); limit lower=-0.698 upper=0.698 effort=10 velocity=1 -> (none); origin xyz=0.14   0.048  0.04 rpy=0  0  0 -> xyz=0.14   0.048  0.035 rpy=0  0  0; type revolute -> fixed
- joint steer_right: axis 0 0 1 -> (none); limit lower=-0.698 upper=0.698 effort=10 velocity=1 -> (none); origin xyz=0.14   -0.048  0.04 rpy=0  0  0 -> xyz=0.14   -0.048  0.035 rpy=0  0  0; type revolute -> fixed

Commit message: fixed bugs in the model. Added ackermann steering skill

File: PiCar-X/simulation/picarx_description/urdf/picarx/picarx.urdf (robot description, URDF)
Before this commit: robot picarx, 8 links, 7 joints
Links:
- removed link picarx_WheelFrontLeft
- removed link picarx_WheelFrontRight
- removed link world
- added link base_link
- added link front_wheel_left, mass 0.025; collision mesh filename=package://picarx_description/meshes/WheelFrontLeft.dae scale=1 1 1; visual mesh filename=package://picarx_description/meshes/WheelFrontLeft.dae scale=1 1 1
- added link front_wheel_right, mass 0.025; collision mesh filename=package://picarx_description/meshes/WheelFrontRight.dae scale=1 1 1; visual mesh filename=package://picarx_description/meshes/WheelFrontRight.dae scale=1 1 1
- link chassis: mass 1 -> 0.350
- link left_wheel: mass 0.1 -> 0.025
- link right_wheel: mass 0.1 -> 0.025
Joints:
- removed joint chassis_to_world
- removed joint front_left_wheel
- removed joint front_right_wheel
- added joint chassis_to_base_link: type fixed, parent base_link, child chassis
- added joint steer_wheel_left: type continuous, parent picarx_steer_fl, child front_wheel_left, origin xyz=0.0 0.012 0.0 rpy=-1.5708 0 0, axis 0  0  1
- added joint steer_wheel_right: type continuous, parent picarx_steer_fr, child front_wheel_right, origin xyz=0.0 -0.012 0.0 rpy=-1.5708 0 0, axis 0  0  1
- joint joint_wheel_left: origin xyz=0 0.055 0.0326 rpy=-1.5708  0 0 -> xyz=0 0.06 0.0326 rpy=-1.5708  0 0
- joint joint_wheel_right: origin xyz=0 -0.055 0.0326 rpy=1.5708  0 0 -> xyz=0 -0.06 0.0326 rpy=1.5708  0 0
- joint steer_left: axis (none) -> 0 0 1; limit (none) -> lower=-0.698132 upper=0.698132 effort=10 velocity=1; type fixed -> revolute
- joint steer_right: axis (none) -> 0 0 1; limit (none) -> lower=-0.698132 upper=0.698132 effort=10 velocity=1; type fixed -> continuous
